File: kicad/ledCAN.kicad_pcb (KiCad board)
At the start: 4 copper layers, 59.7 x 15.2 mm, 43 parts, among them J1 Conn_01x05_MountingPin, J2 Conn_01x04, Q1 PSMQC092N10LS1, Q2 PSMQC076N12LS1, U1 PTCAN11625DMTRQ1, U2 M0A23EC1AC, U3 MPQ4569GQ-AEC1, U4 UCC27282DRCR, U5 NCS214RMUTAG

Commit message: Fix silkscreen mistake, add labeling area
Other:
- board text added: "VOUT PA1 PA0 GND"
- board text removed: "VOUT PA0 PA1 GND"

Commit message: Fix MOSFET footprint mistake
Parts:
- moved C13 11.0 mm to (34.3, 14.2), turned to 180 degrees
- moved R9 6.43 mm to (38.1, 14.2), turned to 180 degrees
- moved Q2 1.63 mm to (36.4, 10.7)
- moved Q1 1.27 mm to (36.3, 5.33), turned to 90 degrees
Connections:
- Q1 pad 1: Net-(Q1-Pad1) -> Net-(C11-Pad2)
- Q1 pad 2: Net-(C11-Pad2) -> Net-(Q1-Pad2)
- Q2 pad 1: Net-(Q2-Pad1) -> GND
- Q2 pad 2: GND -> Net-(Q2-Pad2)
- R7 pad 1: Net-(Q1-Pad1) -> Net-(Q1-Pad2)
- R8 pad 1: Net-(Q2-Pad1) -> Net-(Q2-Pad2)
Routing:
- net Net-(Q1-Pad2): track 0.00 -> 13.1 mm, vias 0 -> 2
- net Net-(C11-Pad2): track 21.2 -> 11.4 mm, vias 54 -> 72
- net Net-(Q2-Pad2): track 0.00 -> 3.95 mm
- net Net-(C15-Pad2): track 9.78 -> 11.6 mm
- net Net-(Q2-Pad1): track 1.64 -> 0.00 mm
- net Net-(Q1-Pad1): track 1.39 -> 0.00 mm
- net GND: track 10.9 -> 12.1 mm, vias 226 -> 227
- net Net-(J2-Pad2): track 32.8 -> 32.0 mm
- net +BATT: vias 38 -> 26
- added copper zone on In2.Cu, net GND
Other:
- board text added: "V1.1"
- board text removed: "V1.0"

Commit message: Change R6 value
Parts:
- R6: value 1.2M -> 1M

Commit message: Update issue date
Other:
- board text added: "City Science @ Taipei Tech Buck converter module with CAN interface DANCHOUZHOU 2022-06 Design in Taiwan Component donated by Nuvoton and PANJIT"
- board text removed: "City Science - MIT Media Lab Buck converter module with CAN interface DANCHOUZHOU 2021-08 Design in Taiwan Component donated by Nuvoton and PANJIT"
Changed lines of the file:
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@@
-(kicad_pcb (version 20171130) (host pcbnew "(5.1.9)-1")
+(kicad_pcb (version 20171130) (host pcbnew 5.0.2+dfsg1-1)
   (general
     (thickness 1.6)
@@
     (34 B.Paste user)
     (35 F.Paste user)
-    (36 B.SilkS user hide)
+    (36 B.SilkS user)
     (37 F.SilkS user)
     (38 B.Mask user)
@@
     (zone_45_only no)
     (trace_min 0.127)
+    (segment_width 0.2)
+    (edge_width 0.05)
     (via_size 0.5)
     (via_drill 0.3)
@@
     (uvia_min_size 0.2)
     (uvia_min_drill 0.1)
-    (edge_width 0.05)
-    (segment_width 0.2)
     (pcb_text_width 0.3)
     (pcb_text_size 1.5 1.5)
@@
     (pad_drill 0.762)
     (pad_to_mask_clearance 0)
+    (solder_mask_min_width 0.25)
     (aux_axis_origin 0 0)
     (visible_elements 7FFFF7FF)
@@
     (effects (font (size 1.5 1.5) (thickness 0.3)) (justify left mirror))
   )
-  (gr_text "City Science - MIT Media Lab\nBuck converter module with CAN interface\nDANCHOUZHOU 2021-08 Design in Taiwan\nComponent donated by Nuvoton and PANJIT" (at 52.324 10.668) (layer B.SilkS)
+  (gr_text "City Science @ Taipei Tech\nBuck converter module with CAN interface\nDANCHOUZHOU 2022-06 Design in Taiwan\nComponent donated by Nuvoton and PANJIT" (at 52.324 10.668) (layer B.SilkS)
     (effects (font (size 1 1) (thickness 0.15)) (justify left mirror))
   )
