File: kicad/ledCAN/ledCAN.kicad_sch (KiCad schematic)
At the start: 0 parts

Commit message: Update page settings
Other:
- company: DANCHOUZHOU -> City Science Lab @ Taipei Tech /a cooperation with the MIT Media Lab
Changed lines of the file:
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@@
   (title_block
     (title "Multi purpose power converter module with CAN bus interface")
-    (date "2021-08-31")
-    (rev "1.1")
-    (company "DANCHOUZHOU")
-    (comment 1 "City Science - MIT Media Lab")
-    (comment 2 "danchouzhou@gmail.com")
+    (date "2022-09-07")
+    (rev "0.1")
+    (company "City Science Lab @ Taipei Tech /a cooperation with the MIT Media Lab")
+    (comment 1 "DANCHOUZHOU")
+    (comment 2 "https://github.com/danchouzhou")
+    (comment 3 "danchouzhou@gmail.com")
   )
   (sheet (at 38.1 25.4) (size 50.8 38.1) (fields_autoplaced)
