File: kicad/ledCAN/TCAN1162x-Q1/PTCAN11625DMTRQ1.kicad_sch (KiCad schematic)
At the start: 7 parts

Commit message: Update page settings
Parts:
- C1: value (none) -> 100nF; footprint (none) -> Capacitor_SMD:C_0603_1608Metric
- C2: value (none) -> 10uF; footprint (none) -> Capacitor_SMD:C_0603_1608Metric
- D1: value (none) -> PEC3124C2A-AU; footprint (none) -> Package_TO_SOT_SMD:SOT-23
- F1: value (none) -> Fuse; footprint (none) -> Fuse:Fuse_1206_3216Metric
- J1: value (none) -> Conn_01x05_MountingPin; footprint (none) -> Connector_JST:JST_PH_S5B-PH-SM4-TB_1x05-1MP_P2.00mm_Horizontal
- R3: value (none) -> 10K; footprint (none) -> Resistor_SMD:R_0603_1608Metric
- U1: value (none) -> PTCAN11625DMTRQ1; footprint (none) -> TI_VSON-14_4.5x3.0mm_DMT0014B:TI_VSON-14_4.5x3.0mm_DMT0014B_ThermalVias
Other:
- company: DANCHOUZHOU -> City Science Lab @ Taipei Tech /a cooperation with the MIT Media Lab
Changed lines of the file:
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@@
   (title_block
     (title "Multi purpose power converter module with CAN bus interface")
-    (date "2021-08-31")
-    (rev "1.1")
-    (company "DANCHOUZHOU")
-    (comment 1 "City Science - MIT Media Lab")
-    (comment 2 "danchouzhou@gmail.com")
+    (date "2022-09-07")
+    (rev "0.1")
+    (company "City Science Lab @ Taipei Tech /a cooperation with the MIT Media Lab")
+    (comment 1 "DANCHOUZHOU")
+    (comment 2 "https://github.com/danchouzhou")
+    (comment 3 "danchouzhou@gmail.com")
   )
   (junction (at 123.19 120.65) (diameter 0) (color 0 0 0 0)
@@
     (in_bom yes) (on_board yes)
     (property "Reference" "U1" (id 0) (at 143.51 83.439 0))
-    (property "Value" "" (id 1) (at 143.51 85.7504 0))
-    (property "Footprint" "" (id 2) (at 143.51 105.41 0)
+    (property "Value" "PTCAN11625DMTRQ1" (id 1) (at 143.51 85.7504 0))
+    (property "Footprint" "TI_VSON-14_4.5x3.0mm_DMT0014B:TI_VSON-14_4.5x3.0mm_DMT0014B_ThermalVias" (id 2) (at 143.51 105.41 0)
       (effects (font (size 1.27 1.27)) hide)
     )
@@
     (in_bom yes) (on_board yes)
     (property "Reference" "D1" (id 0) (at 179.07 99.06 0))
-    (property "Value" "" (id 1) (at 179.07 111.76 0))
-    (property "Footprint" "" (id 2) (at 179.07 88.9 0)
+    (property "Value" "PEC3124C2A-AU" (id 1) (at 179.07 111.76 0))
+    (property "Footprint" "Package_TO_SOT_SMD:SOT-23" (id 2) (at 179.07 88.9 0)
       (effects (font (size 1.27 1.27)) hide)
     )
@@
       (effects (font (size 1.27 1.27)) hide)
     )
-    (property "Value" "" (id 1) (at 165.6588 105.537 90)
+    (property "Value" "GND" (id 1) (at 165.6588 105.537 90)
       (effects (font (size 1.27 1.27)) (justify right))
     )
@@
       (effects (font (size 1.27 1.27)) (justify left))
     )
-    (property "Value" "" (id 1) (at 100.711 125.603 0)
+    (property "Value" "100nF" (id 1) (at 100.711 125.603 0)
       (effects (font (size 1.27 1.27)) (justify left))
     )
-    (property "Footprint" "" (id 2) (at 98.7552 128.27 0)
+    (property "Footprint" "Capacitor_SMD:C_0603_1608Metric" (id 2) (at 98.7552 128.27 0)
       (effects (font (size 1.27 1.27)) hide)
     )
@@
       (effects (font (size 1.27 1.27)) (justify left))
     )
-    (property "Value" "" (id 1) (at 113.411 125.603 0)
+    (property "Value" "10uF" (id 1) (at 113.411 125.603 0)
       (effects (font (size 1.27 1.27)) (justify left))
     )
-    (property "Footprint" "" (id 2) (at 111.4552 128.27 0)
+    (property "Footprint" "Capacitor_SMD:C_0603_1608Metric" (id 2) (at 111.4552 128.27 0)
       (effects (font (size 1.27 1.27)) hide)
     )
@@
       (effects (font (size 1.27 1.27)) hide)
     )
-    (property "Value" "" (id 1) (at 97.917 137.7442 0))
+    (property "Value" "GND" (id 1) (at 97.917 137.7442 0))
     (property "Footprint" "" (id 2) (at 97.79 133.35 0)
       (effects (font (size 1.27 1.27)) hide)
@@
       (effects (font (size 1.27 1.27)) hide)
     )
-    (property "Value" "" (id 1) (at 110.617 137.7442 0))
+    (property "Value" "GND" (id 1) (at 110.617 137.7442 0))
     (property "Footprint" "" (id 2) (at 110.49 133.35 0)
       (effects (font (size 1.27 1.27)) hide)
@@
       (effects (font (size 1.27 1.27)) hide)
     )
-    (property "Value" "" (id 1) (at 123.317 137.7442 0))
+    (property "Value" "GND" (id 1) (at 123.317 137.7442 0))
     (property "Footprint" "" (id 2) (at 123.19 133.35 0)
       (effects (font (size 1.27 1.27)) hide)
@@
       (effects (font (size 1.27 1.27)) hide)
     )
-    (property "Value" "" (id 1) (at 110.871 98.4758 0))
+    (property "Value" "+5V" (id 1) (at 110.871 98.4758 0))
     (property "Footprint" "" (id 2) (at 110.49 102.87 0)
       (effects (font (size 1.27 1.27)) hide)
@@
       (effects (font (size 1.27 1.27)) hide)
     )
-    (property "Value" "" (id 1) (at 98.171 98.4758 0))
+    (property "Value" "+12V" (id 1) (at 98.171 98.4758 0))
     (property "Footprint" "" (id 2) (at 97.79 102.87 0)
       (effects (font (size 1.27 1.27)) hide)
@@
       (effects (font (size 1.27 1.27)) hide)
     )
-    (property "Value" "" (id 1) (at 185.9788 92.837 90)
+    (property "Value" "GND" (id 1) (at 185.9788 92.837 90)
       (effects (font (size 1.27 1.27)) (justify right))
     )
@@
     (in_bom yes) (on_board yes)
     (property "Reference" "F1" (id 0) (at 185.42 85.1662 90))
-    (property "Value" "" (id 1) (at 185.42 87.4776 90))
-    (property "Footprint" "" (id 2) (at 185.42 88.392 90)
+    (property "Value" "Fuse" (id 1) (at 185.42 87.4776 90))
+    (property "Footprint" "Fuse:Fuse_1206_3216Metric" (id 2) (at 185.42 88.392 90)
       (effects (font (size 1.27 1.27)) hide)
     )
@@
       (effects (font (size 1.27 1.27)) hide)
     )
-    (property "Value" "" (id 1) (at 176.911 80.6958 0))
+    (property "Value" "+BATT" (id 1) (at 176.911 80.6958 0))
     (property "Footprint" "" (id 2) (at 176.53 85.09 0)
       (effects (font (size 1.27 1.27)) hide)
@@
       (effects (font (size 1.27 1.27)) hide)
     )
-    (property "Value" "" (id 1) (at 166.751 80.6958 0))
+    (property "Value" "+12V" (id 1) (at 166.751 80.6958 0))
     (property "Footprint" "" (id 2) (at 166.37 85.09 0)
       (effects (font (size 1.27 1.27)) hide)
@@
       (effects (font (size 1.27 1.27)) (justify left))
     )
-    (property "Value" "" (id 1) (at 201.6252 98.4758 0)
+    (property "Value" "Conn_01x05_MountingPin" (id 1) (at 201.6252 98.4758 0)
       (effects (font (size 1.27 1.27)) (justify left))
     )
-    (property "Footprint" "" (id 2) (at 199.39 95.25 0)
+    (property "Footprint" "Connector_JST:JST_PH_S5B-PH-SM4-TB_1x05-1MP_P2.00mm_Horizontal" (id 2) (at 199.39 95.25 0)
       (effects (font (size 1.27 1.27)) hide)
     )
@@
       (effects (font (size 1.27 1.27)) hide)
     )
-    (property "Value" "" (id 1) (at 199.517 114.8842 0))
+    (property "Value" "GND" (id 1) (at 199.517 114.8842 0))
     (property "Footprint" "" (id 2) (at 199.39 110.49 0)
       (effects (font (size 1.27 1.27)) hide)
@@
     (in_bom yes) (on_board yes)
     (property "Reference" "R3" (id 0) (at 119.38 84.9122 90))
-    (property "Value" "" (id 1) (at 119.38 87.2236 90))
-    (property "Footprint" "" (id 2) (at 119.38 88.392 90)
+    (property "Value" "10K" (id 1) (at 119.38 87.2236 90))
+    (property "Footprint" "Resistor_SMD:R_0603_1608Metric" (id 2) (at 119.38 88.392 90)
       (effects (font (size 1.27 1.27)) hide)
     )
@@
       (effects (font (size 1.27 1.27)) hide)
     )
-    (property "Value" "" (id 1) (at 110.617 94.5642 0))
+    (property "Value" "GND" (id 1) (at 110.617 94.5642 0))
     (property "Footprint" "" (id 2) (at 110.49 90.17 0)
       (effects (font (size 1.27 1.27)) hide)
