File: kicad/big-board/M0A21/NuMaker_Volcano.kicad_sch (KiCad schematic)
At the start: 16 parts

Commit message: Update schematic
Parts:
- removed TP? (x3): TestPoint, symbol Connector:TestPoint
- added R?: 330R, symbol Device:R
- added RN? (x2): 4*200R, Resistor_SMD:R_Array_Convex_4x0603, symbol Device:R_Pack04
- added TP? (x2): TP, symbol Connector:TestPoint
- added TP?: RESET, symbol Connector:TestPoint
- added TP? (x2): GND, symbol Connector:TestPoint
- J? (x2): value (none) -> SSQ-107-03-G-D
- R2: value (none) -> 100K
Connections:
- net GND: now also J?.3 (Pin_3), J?.4 (Pin_4), TP?.1, TP?.1
- net PC2: now also RN?.4 (R4.1)
- net PC3: now also RN?.3 (R3.1)
- net PC6: now also RN?.2 (R2.1)
- net PC7: now also RN?.1 (R1.1)
- net PD2: now also R?.1; no longer D?.4 (DIN)
- net PD4: now also RN?.4 (R4.1)
- net PD5: now also RN?.3 (R3.1)
- net PD6: now also RN?.2 (R2.1)
- net PD7: now also RN?.1 (R1.1)
- net TCAN_nRST: now also TP?.1
- net UART0_RXD: now also J?.8 (Pin_8), RN?.7 (R2.2)
- net UART0_TXD: now also J?.10 (Pin_10), RN?.6 (R3.2)
- net VDD: now also J?.1 (Pin_1), J?.2 (Pin_2)
- net USCI0_CTL0: now reaches J?.11 (Pin_11)
- net USCI0_CTL0: now also RN?.8 (R1.2)
- net UART0_CTS: now reaches J?.12 (Pin_12)
- net UART0_CTS: now also RN?.5 (R4.2)
- net USCI0_CLK: now reaches J?.5 (Pin_5)
- net USCI0_CLK: now also RN?.5 (R4.2)
- net UART0_RTS: now reaches J?.6 (Pin_6)
- net UART0_RTS: now also RN?.8 (R1.2)
- net USCI0_DAT1: now reaches J?.7 (Pin_7)
- net USCI0_DAT1: now also RN?.6 (R3.2)
- net USCI0_DAT0: now reaches J?.9 (Pin_9)
- net USCI0_DAT0: now also RN?.7 (R2.2)
- new net: D?.4 (DIN), R?.2
Other:
- note added: "009159010061916 Tin 009159010061911 Flash Gold"
- note added: "1"
- note added: "10"
- note added: "11"
- note added: "12"
- note added: "2"
- note added: "3"
- note added: "4"
- note added: "5"
- note added: "6"
- note added: "7"
- note added: "8"
- note added: "9"
- moved on the sheet: D?

Commit message: Update schematic
Parts:
- added J3: AVX_009159010061, Connector_DebugEdge:DebugEdge_2x05_Target, symbol Connector_Generic:Conn_01x10
- added RN1: 4*200R, Resistor_SMD:R_Array_Convex_4x0603, symbol Device:R_Pack04
- C1, R1: footprint (none) -> Resistor_SMD:R_0603_1608Metric
- C2: renamed from C?; footprint (none) -> Capacitor_SMD:C_0603_1608Metric
- J1: renamed from J?; footprint (none) -> Connector_PinHeader_2.54mm:PinHeader_1x05_P2.54mm_Vertical
- J2, J4: renamed from J?; footprint (none) -> Connector_PinHeader_2.54mm:PinHeader_2x07_P2.54mm_Vertical
- R2, R5: renamed from R?; footprint (none) -> Resistor_SMD:R_0603_1608Metric
- R3: renamed from R2; footprint (none) -> Resistor_SMD:R_0603_1608Metric
- R4: renamed from R3; footprint (none) -> Resistor_SMD:R_0603_1608Metric
- SW1: renamed from SW?; footprint (none) -> Button_Switch_THT:SW_PUSH_6mm
- TP1: renamed from TP?; value RESET -> DATA; footprint (none) -> TestPoint:TestPoint_Keystone_5005-5009_Compact
- TP2: renamed from TP?; value TP -> CLK; footprint (none) -> TestPoint:TestPoint_Keystone_5005-5009_Compact
- TP3: renamed from TP?; value TP -> RST; footprint (none) -> TestPoint:TestPoint_Keystone_5005-5009_Compact
- TP4, TP5: renamed from TP?; footprint (none) -> TestPoint:TestPoint_Keystone_5005-5009_Compact
- U1: renamed from U?; footprint (none) -> Package_SO:TSSOP-28_4.4x9.7mm_P0.65mm
- gave numbers to parts that had none: 4
Connections:
- net GND: now also J3.8 (Pin_8)
- net IO_PA0: now also TP1.1, RN1.5 (R4.2)
- net IO_PA1: now also TP2.1, RN1.8 (R1.2)
- net PB4: now also RN1.6 (R3.2)
- net PB6: now also RN1.7 (R2.2)
- net TCAN_nRST: now also R2.1, SW1.2, J3.6 (Pin_6); no longer C1.1, J1.4 (Pin_4), J2.4 (Pin_4), R1.1, R2.2, TP1.1, U1.4 (PA3)
- net PA3: now reaches TP3.1
- net PA3: now also C1.1, J1.4 (Pin_4), J2.4 (Pin_4), R1.1, R2.2, U1.4 (PA3)
- new net: J3.5 (Pin_5), RN1.1 (R1.1)
- new net: J3.4 (Pin_4), RN1.2 (R2.1)
- new net: J3.3 (Pin_3), RN1.3 (R3.1)
- new net: J3.2 (Pin_2), RN1.4 (R4.1)
- no-connect marks 1 -> 5
Other:
- note added: "AVX-KYOCERA BTB 00-9159 009159010061916 Tin 009159010061911 Flash Gold"
- note added: "CLK"
- note added: "GND"
- note added: "RST"
- note added: "RXD"
- note added: "STLINK-V3MINIE"
- note added: "TDI"
- note added: "TDO"
- note added: "TMS"
- note added: "TXD"
- note added: "VCC"
- note removed: "009159010061916 Tin 009159010061911 Flash Gold"
- title: Evaluation board of ledCAN -> Multi purpose power converter module with CAN bus interface
- moved on the sheet: C2, TP1, TP2, TP3, TP4, TP5, U1

Commit message: Update PCB
Connections:
- net IO_PA0: now also RN1.8 (R1.2); no longer RN1.5 (R4.2)
- net IO_PA1: now also RN1.5 (R4.2); no longer RN1.8 (R1.2)
- net PB4: now also RN1.7 (R2.2); no longer RN1.6 (R3.2)
- net PB6: now also RN1.6 (R3.2); no longer RN1.7 (R2.2)
- net PC2: now also RN3.2 (R2.1); no longer RN2.4 (R4.1)
- net PC3: now also RN3.4 (R4.1); no longer RN2.3 (R3.1)
- net PC7: now also RN2.4 (R4.1); no longer RN2.1 (R1.1)
- net PD4: now also RN2.3 (R3.1); no longer RN3.4 (R4.1)
- net PD5: now also RN2.1 (R1.1); no longer RN3.3 (R3.1)
- net PD6: now also RN3.3 (R3.1); no longer RN3.2 (R2.1)
- net UART0_CTS: now also RN3.7 (R2.2); no longer RN2.5 (R4.2)
- net UART0_RTS: now also RN2.5 (R4.2); no longer RN2.8 (R1.2)
- net UART0_TXD: now also RN3.5 (R4.2); no longer RN2.6 (R3.2)
- net USCI0_CLK: now also RN2.6 (R3.2); no longer RN3.5 (R4.2)
- net USCI0_DAT0: now also RN3.6 (R3.2); no longer RN3.7 (R2.2)
- net USCI0_DAT1: now also RN2.8 (R1.2); no longer RN3.6 (R3.2)
- net at RN1.1 (R1.1): now also J3.2 (Pin_2); no longer J3.5 (Pin_5)
- net at RN1.2 (R2.1): now also J3.3 (Pin_3); no longer J3.4 (Pin_4)
- net at RN1.3 (R3.1): now also J3.4 (Pin_4); no longer J3.3 (Pin_3)
- net at RN1.4 (R4.1): now also J3.5 (Pin_5); no longer J3.2 (Pin_2)
Changed lines of the file:
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@@
     (effects (font (size 1.27 1.27)) (justify left bottom))
   )
-  (label "PD5" (at 259.08 106.68 180)
+  (label "PD5" (at 259.08 93.98 180)
     (effects (font (size 1.27 1.27)) (justify right bottom))
   )
@@
     (effects (font (size 1.27 1.27)) (justify right bottom))
   )
-  (label "PC2" (at 259.08 86.36 180)
+  (label "PC2" (at 259.08 109.22 180)
     (effects (font (size 1.27 1.27)) (justify right bottom))
   )
@@
     (effects (font (size 1.27 1.27)) (justify left bottom))
   )
-  (label "PC7" (at 259.08 93.98 180)
+  (label "PC7" (at 259.08 86.36 180)
     (effects (font (size 1.27 1.27)) (justify right bottom))
   )
@@
     (effects (font (size 1.27 1.27)) (justify right bottom))
   )
-  (label "PC3" (at 259.08 88.9 180)
+  (label "PC3" (at 259.08 104.14 180)
     (effects (font (size 1.27 1.27)) (justify right bottom))
   )
@@
     (effects (font (size 1.27 1.27)) (justify left bottom))
   )
-  (label "UART0_RTS" (at 226.06 93.98 0)
+  (label "UART0_RTS" (at 226.06 86.36 0)
     (effects (font (size 1.27 1.27)) (justify left bottom))
   )
@@
     (effects (font (size 1.27 1.27)) (justify right bottom))
   )
-  (label "UART0_TXD" (at 226.06 88.9 0)
+  (label "UART0_TXD" (at 226.06 104.14 0)
     (effects (font (size 1.27 1.27)) (justify left bottom))
   )
@@
     (effects (font (size 1.27 1.27)) (justify left bottom))
   )
-  (label "PD4" (at 259.08 104.14 180)
+  (label "PD4" (at 259.08 88.9 180)
     (effects (font (size 1.27 1.27)) (justify right bottom))
   )
@@
     (effects (font (size 1.27 1.27)) (justify right bottom))
   )
-  (label "USCI0_DAT1" (at 226.06 106.68 0)
+  (label "USCI0_DAT1" (at 226.06 93.98 0)
     (effects (font (size 1.27 1.27)) (justify left bottom))
   )
@@
     (effects (font (size 1.27 1.27)) (justify left bottom))
   )
-  (label "USCI0_CLK" (at 226.06 104.14 0)
+  (label "USCI0_CLK" (at 226.06 88.9 0)
     (effects (font (size 1.27 1.27)) (justify left bottom))
   )
@@
     (effects (font (size 1.27 1.27)) (justify left bottom))
   )
-  (label "UART0_CTS" (at 226.06 86.36 0)
+  (label "UART0_CTS" (at 226.06 109.22 0)
     (effects (font (size 1.27 1.27)) (justify left bottom))
   )
@@
     (effects (font (size 1.27 1.27)) (justify left bottom))
   )
-  (label "USCI0_DAT0" (at 226.06 109.22 0)
-    (effects (font (size 1.27 1.27)) (justify left bottom))
-  )
-  (label "PD6" (at 259.08 109.22 180)
+  (label "USCI0_DAT0" (at 226.06 106.68 0)
+    (effects (font (size 1.27 1.27)) (justify left bottom))
+  )
+  (label "PD6" (at 259.08 106.68 180)
     (effects (font (size 1.27 1.27)) (justify right bottom))
   )
@@
     (pin "1")
   )
-  (symbol (lib_id "Device:R_Pack04") (at 107.95 93.98 90) (unit 1)
+  (symbol (lib_id "Device:R_Pack04") (at 107.95 96.52 90) (mirror x) (unit 1)
     (in_bom yes) (on_board yes) (fields_autoplaced)
     (property "Reference" "RN1" (id 0) (at 107.95 85.09 90))
     (property "Value" "4*200R" (id 1) (at 107.95 87.63 90))
-    (property "Footprint" "Resistor_SMD:R_Array_Convex_4x0603" (id 2) (at 107.95 86.995 90)
-      (effects (font (size 1.27 1.27)) hide)
-    )
-    (property "Datasheet" "~" (id 3) (at 107.95 93.98 0)
-      (effects (font (size 1.27 1.27)) hide)
-    )
+    (property "Footprint" "Resistor_SMD:R_Array_Convex_4x0603" (id 2) (at 107.95 103.505 90)
+      (effects (font (size 1.27 1.27)) hide)
+    )
+    (property "Datasheet" "~" (id 3) (at 107.95 96.52 0)
+      (effects (font (size 1.27 1.27)) hide)
+    )
