File: kicad/big-board/MPQ4569/MPQ4569GQ-AEC1-Z.kicad_sch (KiCad schematic)
At the start: 10 parts

Commit message: Update schematic
Parts:
- C?: value (none) -> 10nF; footprint (none) -> Capacitor_SMD:C_0603_1608Metric
- C?: value (none) -> 10uF; footprint (none) -> Capacitor_SMD:C_0805_2012Metric
- C?: value (none) -> 10uF; footprint (none) -> Capacitor_SMD:C_1210_3225Metric
- C?: value (none) -> 100nF; footprint (none) -> Capacitor_SMD:C_0603_1608Metric
- C?: value (none) -> 39pF; footprint (none) -> Capacitor_SMD:C_0603_1608Metric
- L?: value (none) -> TYA252012100M-10; footprint (none) -> tya252010-series:tya252010-series
- R? (x2): value (none) -> 1M; footprint (none) -> Resistor_SMD:R_0603_1608Metric
- R?: value (none) -> 91K; footprint (none) -> Resistor_SMD:R_0603_1608Metric
- U?: value (none) -> MPQ4569GQ-AEC1; footprint (none) -> QFN-10-1EP_3x3mm_P0.5mm_EP1.7x2.5mm:QFN-10-1EP_3x3mm_P0.5mm_EP1.7x2.5mm
Changed lines of the file:
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@@
     (in_bom yes) (on_board yes)
     (property "Reference" "U?" (id 0) (at 139.7 100.33 0))
-    (property "Value" "" (id 1) (at 139.7 102.87 0))
-    (property "Footprint" "" (id 2) (at 139.7 68.58 0)
+    (property "Value" "MPQ4569GQ-AEC1" (id 1) (at 139.7 102.87 0))
+    (property "Footprint" "QFN-10-1EP_3x3mm_P0.5mm_EP1.7x2.5mm:QFN-10-1EP_3x3mm_P0.5mm_EP1.7x2.5mm" (id 2) (at 139.7 68.58 0)
       (effects (font (size 1.27 1.27)) hide)
     )
@@
       (effects (font (size 1.27 1.27)) (justify left))
     )
-    (property "Value" "" (id 1) (at 123.698 84.963 0)
-      (effects (font (size 1.27 1.27)) (justify left))
-    )
-    (property "Footprint" "" (id 2) (at 120.142 83.82 90)
+    (property "Value" "1M" (id 1) (at 123.698 84.963 0)
+      (effects (font (size 1.27 1.27)) (justify left))
+    )
+    (property "Footprint" "Resistor_SMD:R_0603_1608Metric" (id 2) (at 120.142 83.82 90)
       (effects (font (size 1.27 1.27)) hide)
     )
@@
     (in_bom yes) (on_board yes)
     (property "Reference" "C?" (id 0) (at 118.11 121.8692 90))
-    (property "Value" "" (id 1) (at 118.11 124.1806 90))
-    (property "Footprint" "" (id 2) (at 114.3 129.2352 0)
+    (property "Value" "10nF" (id 1) (at 118.11 124.1806 90))
+    (property "Footprint" "Capacitor_SMD:C_0603_1608Metric" (id 2) (at 114.3 129.2352 0)
       (effects (font (size 1.27 1.27)) hide)
     )
@@
       (effects (font (size 1.27 1.27)) hide)
     )
-    (property "Value" "" (id 1) (at 109.347 132.6642 0))
+    (property "Value" "GND" (id 1) (at 109.347 132.6642 0))
     (property "Footprint" "" (id 2) (at 109.22 128.27 0)
       (effects (font (size 1.27 1.27)) hide)
@@
       (effects (font (size 1.27 1.27)) hide)
     )
-    (property "Value" "" (id 1) (at 138.557 147.9042 0))
+    (property "Value" "GND" (id 1) (at 138.557 147.9042 0))
     (property "Footprint" "" (id 2) (at 138.43 143.51 0)
       (effects (font (size 1.27 1.27)) hide)
@@
       (effects (font (size 1.27 1.27)) (justify left))
     )
-    (property "Value" "" (id 1) (at 198.501 84.963 0)
-      (effects (font (size 1.27 1.27)) (justify left))
-    )
-    (property "Footprint" "" (id 2) (at 196.5452 87.63 0)
+    (property "Value" "10uF" (id 1) (at 198.501 84.963 0)
+      (effects (font (size 1.27 1.27)) (justify left))
+    )
+    (property "Footprint" "Capacitor_SMD:C_0805_2012Metric" (id 2) (at 196.5452 87.63 0)
       (effects (font (size 1.27 1.27)) hide)
     )
@@
       (effects (font (size 1.27 1.27)) hide)
     )
-    (property "Value" "" (id 1) (at 195.707 97.1042 0))
+    (property "Value" "GND" (id 1) (at 195.707 97.1042 0))
     (property "Footprint" "" (id 2) (at 195.58 92.71 0)
       (effects (font (size 1.27 1.27)) hide)
@@
       (effects (font (size 1.27 1.27)) hide)
     )
-    (property "Value" "" (id 1) (at 195.961 65.4558 0))
+    (property "Value" "+12V" (id 1) (at 195.961 65.4558 0))
     (property "Footprint" "" (id 2) (at 195.58 69.85 0)
       (effects (font (size 1.27 1.27)) hide)
@@
       (effects (font (size 1.27 1.27)) (justify left))
     )
-    (property "Value" "" (id 1) (at 114.681 84.963 0)
-      (effects (font (size 1.27 1.27)) (justify left))
-    )
-    (property "Footprint" "" (id 2) (at 112.7252 87.63 0)
+    (property "Value" "10uF" (id 1) (at 114.681 84.963 0)
+      (effects (font (size 1.27 1.27)) (justify left))
+    )
+    (property "Footprint" "Capacitor_SMD:C_1210_3225Metric" (id 2) (at 112.7252 87.63 0)
       (effects (font (size 1.27 1.27)) hide)
     )
@@
       (effects (font (size 1.27 1.27)) hide)
     )
-    (property "Value" "" (id 1) (at 111.887 97.1042 0))
+    (property "Value" "GND" (id 1) (at 111.887 97.1042 0))
     (property "Footprint" "" (id 2) (at 111.76 92.71 0)
       (effects (font (size 1.27 1.27)) hide)
@@
     (in_bom yes) (on_board yes)
     (property "Reference" "L?" (id 0) (at 171.45 69.215 90))
-    (property "Value" "" (id 1) (at 171.45 71.5264 90))
-    (property "Footprint" "" (id 2) (at 171.45 74.93 0)
+    (property "Value" "TYA252012100M-10" (id 1) (at 171.45 71.5264 90))
+    (property "Footprint" "tya252010-series:tya252010-series" (id 2) (at 171.45 74.93 0)
       (effects (font (size 1.27 1.27)) hide)
     )
@@
     (in_bom yes) (on_board yes)
     (property "Reference" "C?" (id 0) (at 148.59 58.3692 90))
-    (property "Value" "" (id 1) (at 148.59 60.6806 90))
-    (property "Footprint" "" (id 2) (at 144.78 65.7352 0)
+    (property "Value" "100nF" (id 1) (at 148.59 60.6806 90))
+    (property "Footprint" "Capacitor_SMD:C_0603_1608Metric" (id 2) (at 144.78 65.7352 0)
       (effects (font (size 1.27 1.27)) hide)
     )
@@
     (in_bom yes) (on_board yes)
     (property "Reference" "R?" (id 0) (at 176.53 106.5022 90))
-    (property "Value" "" (id 1) (at 176.53 108.8136 90))
-    (property "Footprint" "" (id 2) (at 176.53 109.982 90)
+    (property "Value" "1M" (id 1) (at 176.53 108.8136 90))
+    (property "Footprint" "Resistor_SMD:R_0603_1608Metric" (id 2) (at 176.53 109.982 90)
       (effects (font (size 1.27 1.27)) hide)
     )
@@
     (in_bom yes) (on_board yes)
     (property "Reference" "C?" (id 0) (at 176.53 115.5192 90))
-    (property "Value" "" (id 1) (at 176.53 117.8306 90))
-    (property "Footprint" "" (id 2) (at 172.72 122.8852 0)
+    (property "Value" "39pF" (id 1) (at 176.53 117.8306 90))
+    (property "Footprint" "Capacitor_SMD:C_0603_1608Metric" (id 2) (at 172.72 122.8852 0)
       (effects (font (size 1.27 1.27)) hide)
     )
@@
       (effects (font (size 1.27 1.27)) (justify left))
     )
-    (property "Value" "" (id 1) (at 159.258 121.793 0)
-      (effects (font (size 1.27 1.27)) (justify left))
-    )
-    (property "Footprint" "" (id 2) (at 155.702 120.65 90)
+    (property "Value" "91K" (id 1) (at 159.258 121.793 0)
+      (effects (font (size 1.27 1.27)) (justify left))
+    )
+    (property "Footprint" "Resistor_SMD:R_0603_1608Metric" (id 2) (at 155.702 120.65 90)
       (effects (font (size 1.27 1.27)) hide)
     )
@@
       (effects (font (size 1.27 1.27)) hide)
     )
-    (property "Value" "" (id 1) (at 157.607 133.9342 0))
+    (property "Value" "GND" (id 1) (at 157.607 133.9342 0))
     (property "Footprint" "" (id 2) (at 157.48 129.54 0)
       (effects (font (size 1.27 1.27)) hide)

Commit message: Update schematic
Parts:
- gave numbers to parts that had none: 10
Changed lines of the file:
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@@
     (rev "0.1")
     (company "City Science Lab @ Taipei Tech /a cooperation with the MIT Media Lab")
-    (comment 1 "DANCHOUZHOU")
+    (comment 1 "DANCHOUZHOU © Danny Chou, all rights reserved.")
     (comment 2 "https://github.com/danchouzhou")
     (comment 3 "danchouzhou@gmail.com")
@@
   (symbol (lib_id "MPQ4569:MPQ4569GQ-AEC1") (at 139.7 101.6 0) (unit 1)
     (in_bom yes) (on_board yes)
-    (property "Reference" "U?" (id 0) (at 139.7 100.33 0))
+    (property "Reference" "U3" (id 0) (at 139.7 100.33 0))
     (property "Value" "MPQ4569GQ-AEC1" (id 1) (at 139.7 102.87 0))
     (property "Footprint" "QFN-10-1EP_3x3mm_P0.5mm_EP1.7x2.5mm:QFN-10-1EP_3x3mm_P0.5mm_EP1.7x2.5mm" (id 2) (at 139.7 68.58 0)
@@
   (symbol (lib_id "Device:R") (at 121.92 83.82 0) (unit 1)
     (in_bom yes) (on_board yes)
-    (property "Reference" "R?" (id 0) (at 123.698 82.6516 0)
+    (property "Reference" "R11" (id 0) (at 123.698 82.6516 0)
       (effects (font (size 1.27 1.27)) (justify left))
     )
@@
   (symbol (lib_id "Device:C") (at 118.11 128.27 270) (unit 1)
     (in_bom yes) (on_board yes)
-    (property "Reference" "C?" (id 0) (at 118.11 121.8692 90))
+    (property "Reference" "C9" (id 0) (at 118.11 121.8692 90))
     (property "Value" "10nF" (id 1) (at 118.11 124.1806 90))
     (property "Footprint" "Capacitor_SMD:C_0603_1608Metric" (id 2) (at 114.3 129.2352 0)
@@
   (symbol (lib_id "power:GND") (at 109.22 128.27 0) (unit 1)
     (in_bom yes) (on_board yes)
-    (property "Reference" "#PWR?" (id 0) (at 109.22 134.62 0)
+    (property "Reference" "#PWR040" (id 0) (at 109.22 134.62 0)
       (effects (font (size 1.27 1.27)) hide)
     )
@@
   (symbol (lib_id "power:GND") (at 138.43 143.51 0) (unit 1)
     (in_bom yes) (on_board yes)
-    (property "Reference" "#PWR?" (id 0) (at 138.43 149.86 0)
+    (property "Reference" "#PWR042" (id 0) (at 138.43 149.86 0)
       (effects (font (size 1.27 1.27)) hide)
     )
@@
   (symbol (lib_id "Device:C") (at 195.58 83.82 0) (unit 1)
     (in_bom yes) (on_board yes)
-    (property "Reference" "C?" (id 0) (at 198.501 82.6516 0)
+    (property "Reference" "C12" (id 0) (at 198.501 82.6516 0)
       (effects (font (size 1.27 1.27)) (justify left))
     )
@@
   (symbol (lib_id "power:GND") (at 195.58 92.71 0) (unit 1)
     (in_bom yes) (on_board yes)
-    (property "Reference" "#PWR?" (id 0) (at 195.58 99.06 0)
+    (property "Reference" "#PWR045" (id 0) (at 195.58 99.06 0)
       (effects (font (size 1.27 1.27)) hide)
     )
@@
   (symbol (lib_id "power:+12V") (at 195.58 69.85 0) (unit 1)
     (in_bom yes) (on_board yes)
-    (property "Reference" "#PWR?" (id 0) (at 195.58 73.66 0)
+    (property "Reference" "#PWR044" (id 0) (at 195.58 73.66 0)
       (effects (font (size 1.27 1.27)) hide)
     )
@@
   (symbol (lib_id "Device:C") (at 111.76 83.82 0) (unit 1)
     (in_bom yes) (on_board yes)
-    (property "Reference" "C?" (id 0) (at 114.681 82.6516 0)
+    (property "Reference" "C8" (id 0) (at 114.681 82.6516 0)
       (effects (font (size 1.27 1.27)) (justify left))
     )
@@
   (symbol (lib_id "power:+BATT") (at 106.68 74.93 0) (unit 1)
     (in_bom yes) (on_board yes)
-    (property "Reference" "#PWR?" (id 0) (at 106.68 78.74 0)
+    (property "Reference" "#PWR039" (id 0) (at 106.68 78.74 0)
       (effects (font (size 1.27 1.27)) hide)
     )
@@
   (symbol (lib_id "power:GND") (at 111.76 92.71 0) (unit 1)
     (in_bom yes) (on_board yes)
-    (property "Reference" "#PWR?" (id 0) (at 111.76 99.06 0)
+    (property "Reference" "#PWR041" (id 0) (at 111.76 99.06 0)
       (effects (font (size 1.27 1.27)) hide)
     )
@@
   (symbol (lib_id "Device:L_Iron") (at 171.45 74.93 90) (unit 1)
     (in_bom yes) (on_board yes)
-    (property "Reference" "L?" (id 0) (at 171.45 69.215 90))
+    (property "Reference" "L1" (id 0) (at 171.45 69.215 90))
     (property "Value" "TYA252012100M-10" (id 1) (at 171.45 71.5264 90))
     (property "Footprint" "tya252010-series:tya252010-series" (id 2) (at 171.45 74.93 0)
@@
   (symbol (lib_id "Device:C") (at 148.59 64.77 270) (unit 1)
     (in_bom yes) (on_board yes)
-    (property "Reference" "C?" (id 0) (at 148.59 58.3692 90))
+    (property "Reference" "C10" (id 0) (at 148.59 58.3692 90))
     (property "Value" "100nF" (id 1) (at 148.59 60.6806 90))
     (property "Footprint" "Capacitor_SMD:C_0603_1608Metric" (id 2) (at 144.78 65.7352 0)
@@
   (symbol (lib_id "Device:R") (at 176.53 111.76 270) (unit 1)
     (in_bom yes) (on_board yes)
-    (property "Reference" "R?" (id 0) (at 176.53 106.5022 90))
+    (property "Reference" "R13" (id 0) (at 176.53 106.5022 90))
     (property "Value" "1M" (id 1) (at 176.53 108.8136 90))
     (property "Footprint" "Resistor_SMD:R_0603_1608Metric" (id 2) (at 176.53 109.982 90)
@@
   (symbol (lib_id "Device:C") (at 176.53 121.92 270) (unit 1)
     (in_bom yes) (on_board yes)
-    (property "Reference" "C?" (id 0) (at 176.53 115.5192 90))
+    (property "Reference" "C11" (id 0) (at 176.53 115.5192 90))
     (property "Value" "39pF" (id 1) (at 176.53 117.8306 90))
     (property "Footprint" "Capacitor_SMD:C_0603_1608Metric" (id 2) (at 172.72 122.8852 0)
@@
   (symbol (lib_id "Device:R") (at 157.48 120.65 0) (unit 1)
     (in_bom yes) (on_board yes)
-    (property "Reference" "R?" (id 0) (at 159.258 119.4816 0)
+    (property "Reference" "R12" (id 0) (at 159.258 119.4816 0)
       (effects (font (size 1.27 1.27)) (justify left))
     )
@@
   (symbol (lib_id "power:GND") (at 157.48 129.54 0) (unit 1)
     (in_bom yes) (on_board yes)
-    (property "Reference" "#PWR?" (id 0) (at 157.48 135.89 0)
-      (effects (font (size 1.27 1.27)) hide)
-    )
+    (property "Reference" "#PWR043" (id 0) (at 157.48 135.89 0)
+      (effects (font (size 1.27 1.27)) hide)
+    )

Commit message: Update PCB
Parts:
- added TP15: VDD, TestPoint:TestPoint_Keystone_5005-5009_Compact, symbol Connector:TestPoint
- added TP16: 12V, TestPoint:TestPoint_Keystone_5005-5009_Compact, symbol Connector:TestPoint
- added TP17: VBAT, TestPoint:TestPoint_Keystone_5005-5009_Compact, symbol Connector:TestPoint
- added TP18, TP19, TP20: GND, TestPoint:TestPoint_Keystone_5005-5009_Compact, symbol Connector:TestPoint
Connections:
- net +12V: now also TP16.1
- net +BATT: now also TP17.1
- net GND: now also TP18.1, TP19.1, TP20.1
- new net VDD: TP15.1
Other:
- note added: "Power input"
