File: kicad/big-board/TCAN1162x-Q1/PTCAN11625DMTRQ1.kicad_sch (KiCad schematic)
At the start: 13 parts

Commit message: Update schematic
Parts:
- added J?: Conn_02x05_Odd_Even, symbol Connector_Generic:Conn_02x05_Odd_Even
- added R? (x2): 330R, symbol Device:R
- D?: value (none) -> PEC3124C2A-AU; footprint (none) -> Package_TO_SOT_SMD:SOT-23
- U?: value (none) -> PTCAN11625DMTRQ1; footprint (none) -> TI_VSON-14_4.5x3.0mm_DMT0014B:TI_VSON-14_4.5x3.0mm_DMT0014B_ThermalVias
Connections:
- net GND: now also J?.2 (Pin_2), J?.4 (Pin_4), J?.5 (Pin_5), J?.7 (Pin_7), J?.9 (Pin_9)
- net INH: now also J?.3 (Pin_3)
- net TCAN_TS: now also J?.10 (Pin_10)
- net TCAN_nRST: now also R?.2; no longer U?.11 (nRST)
- net TCAN_nSLP: now also R?.2; no longer U?.14 (nSLP)
- net WAKE: now also J?.1 (Pin_1)
- new net nRST: J?.6 (Pin_6), R?.1, U?.11 (nRST)
- new net nSLP: J?.8 (Pin_8), R?.1, U?.14 (nSLP)
Other:
- moved on the sheet: J?

Commit message: Update schematic
Parts:
- C3, C4, C7: renamed from C?; footprint (none) -> Capacitor_SMD:C_0603_1608Metric
- C5, C6: renamed from C?; footprint (none) -> Resistor_SMD:R_0805_2012Metric
- J6: renamed from J?; footprint (none) -> Connector_PinHeader_2.54mm:PinHeader_2x05_P2.54mm_Vertical
- J7: renamed from J?; footprint (none) -> Connector_PinHeader_2.54mm:PinHeader_1x03_P2.54mm_Vertical
- J8: renamed from J?; footprint (none) -> Connector_PinHeader_2.54mm:PinHeader_1x02_P2.54mm_Vertical
- R10, R6, R7, R9: renamed from R?; footprint (none) -> Resistor_SMD:R_0603_1608Metric
- R8: renamed from R?; footprint (none) -> Resistor_SMD:R_1206_3216Metric
- SW2: renamed from SW?; footprint (none) -> Button_Switch_THT:SW_PUSH_6mm
- gave numbers to parts that had none: 2
Other:
- note added: "Opt. for TCAN11623"

Commit message: Update PCB
Connections:
- net +3.3V: now also J7.1 (Pin_1); no longer J7.3 (Pin_3)
- net +5V: now also J7.3 (Pin_3); no longer J7.1 (Pin_1)
Changed lines of the file:
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@@
     (pin "1")
   )
-  (symbol (lib_id "Connector_Generic:Conn_01x03") (at 55.88 97.79 0) (unit 1)
+  (symbol (lib_id "Connector_Generic:Conn_01x03") (at 55.88 97.79 0) (mirror x) (unit 1)
     (in_bom yes) (on_board yes) (fields_autoplaced)
-    (property "Reference" "J7" (id 0) (at 58.42 96.5199 0)
-      (effects (font (size 1.27 1.27)) (justify left))
-    )
-    (property "Value" "VDD_SEL" (id 1) (at 58.42 99.0599 0)
-      (effects (font (size 1.27 1.27)) (justify left))
-    )
+    (property "Reference" "J7" (id 0) (at 55.88 88.9 0))
+    (property "Value" "VDD_SEL" (id 1) (at 55.88 91.44 0))
     (property "Footprint" "Connector_PinHeader_2.54mm:PinHeader_1x03_P2.54mm_Vertical" (id 2) (at 55.88 97.79 0)
       (effects (font (size 1.27 1.27)) hide)
