File: kicad/big-board/ledCAN_bigBoard.kicad_pcb (KiCad board)
At the start: 2 copper layers, 127.3 x 63.5 mm, 92 parts, among them J1 Nu-Link, J2 SSQ-107-03-G-D, J3 AVX_009159010061, J4 SSQ-107-03-G-D, J5 Pmod, J6 Conn_02x05_Odd_Even, J7 VDD_SEL, J8 CAN_bus, J9 Conn_01x04, Q1 PSMQC092N10LS1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

Commit message: Update PCB
Parts:
- C16: footprint Capacitor_SMD:C_0805_2012Metric_Pad1.18x1.45mm_HandSolder -> Capacitor_SMD:C_1206_3216Metric
- R16: footprint Resistor_SMD:R_0805_2012Metric -> Resistor_SMD:R_1206_3216Metric_Pad1.30x1.75mm_HandSolder
- moved J6 91.6 mm to (167.6, 49.5)
- moved C3 91.6 mm to (177.5, 24.4)
- moved R6 91.6 mm to (187.6, 24.9)
- moved R7 91.6 mm to (182.6, 24.4)
- moved J7 89.8 mm to (72.6, 27.9), turned to 90 degrees
- moved SW1 87.1 mm to (109.8, 55.5)
- moved J1 78.9 mm to (92.4, 53.3), turned to -90 degrees
- moved TP7 78.1 mm to (111.8, 29.2)
- moved C5 77.4 mm to (76.2, 33.4), turned to 90 degrees
- moved C7 76.0 mm to (73.7, 33.6), turned to 90 degrees
- moved U2 69.4 mm to (75.2, 39.0), turned to -90 degrees
- moved C1 66.2 mm to (102.5, 33.7)
- moved R1 64.4 mm to (102.5, 37.5), turned to 180 degrees
- moved R2 63.6 mm to (102.5, 39.4)
- moved C4 62.0 mm to (73.9, 44.6), turned to -90 degrees
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Connections:
- J7 pad 1: +5V -> +3.3V
- J7 pad 3: +3.3V -> +5V
Routing:
- net /MCU/PA3: track 5.92 -> 49.9 mm, vias 0 -> 3
- net VDD: track 13.4 -> 52.8 mm, vias 0 -> 2
- net GND: track 6.16 -> 38.5 mm, vias 0 -> 5
- net TCAN_RXD: track 7.03 -> 32.8 mm, vias 0 -> 2
- net TCAN_TXD: track 5.41 -> 26.3 mm, vias 0 -> 2
- net IO_PA1: track 15.0 -> 30.6 mm, vias 0 -> 1
- net IO_PA0: track 17.3 -> 30.8 mm, vias 2 -> 3
- net +3.3V: track 3.52 -> 16.9 mm
- net +5V: track 0.00 -> 10.9 mm
- net /CAN Transceiver/nRST: track 0.00 -> 7.81 mm, vias 0 -> 2
- net /MCU/PD5: track 29.6 -> 22.8 mm, vias 1 -> 2
- net /MCU/PD4: track 34.8 -> 28.5 mm, vias 1 -> 2
- net /MCU/PC7: track 17.0 -> 21.2 mm, vias 0 -> 3
- net /MCU/PC3: track 33.6 -> 30.0 mm
- net /MCU/PD6: track 30.4 -> 27.0 mm
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Other:
- board size 127.3 x 63.5 mm -> 127 x 63.5 mm
- board text added: "GND"
- board text added: "PC2"
- board text added: "PC3"
- board text added: "PC6"
- board text added: "PC7"
- board text added: "PD4"
- board text added: "PD5"
- board text added: "PD6"
- board text added: "PD7"
- board text added: "Pmod"
- board text added: "VDD"

Commit message: Update PCB
Parts:
- moved R17 227.0 mm to (135.5, 34.2)
- moved R18 227.0 mm to (135.5, 36.7)
- moved J9 227.0 mm to (141.2, 35.3)
- moved TP15 208.4 mm to (146.1, 15.3)
- moved TP18 208.4 mm to (156.2, 20.3)
- moved TP19 208.4 mm to (156.2, 15.3)
- moved TP20 208.4 mm to (146.1, 20.3)
- moved TP16 208.4 mm to (151.2, 20.3)
- moved TP17 208.4 mm to (151.2, 15.3)
- moved C18 173.4 mm to (93.7, 22.1)
- moved U5 171.0 mm to (97.0, 22.2), turned to 180 degrees
- moved R6 129.7 mm to (59.7, 46.2), turned to 180 degrees
- moved R7 124.5 mm to (59.7, 44.2)
- moved C3 119.1 mm to (59.7, 42.2), turned to 180 degrees
- moved J6 104.0 mm to (64.3, 38.4), turned to 0 degrees
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Connections:
- R19 pad 1: Net-(L2-Pad2) -> Net-(R19-Pad1)
- R19 pad 3: Net-(R19-Pad3) -> Net-(L2-Pad2)
- U5 pad 4: Net-(R19-Pad3) -> Net-(R19-Pad1)
- U5 pad 5: Net-(R19-Pad3) -> Net-(R19-Pad1)
Routing:
- net VDD: track 52.8 -> 100.7 mm, vias 2 -> 6
- net SYNC_VFB: track 5.14 -> 30.9 mm, vias 0 -> 4
- net /CAN Transceiver/WAKE: track 0.00 -> 23.2 mm, vias 0 -> 3
- net TCAN_TS: track 11.7 -> 31.2 mm, vias 1 -> 3
- net /CAN Transceiver/nRST: track 7.81 -> 23.5 mm, vias 2 -> 5
- net /CAN Transceiver/INH: track 0.00 -> 13.7 mm, vias 0 -> 3
- net /CAN Transceiver/nSLP: track 3.03 -> 15.4 mm, vias 0 -> 1
- net Net-(R19-Pad2): track 0.00 -> 5.52 mm
- net Net-(R19-Pad1): track 0.00 -> 5.48 mm
- net IO_PA1: track 30.6 -> 34.9 mm, vias 1 -> 2
- net IO_PA0: track 30.8 -> 34.8 mm, vias 3 -> 4
- net Net-(C11-Pad2): track 0.00 -> 3.73 mm
- net Net-(C9-Pad1): track 0.00 -> 3.71 mm
- net Net-(D1-Pad4): track 0.00 -> 2.57 mm
- net Net-(Q2-Pad2): track 0.00 -> 2.50 mm
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- added copper zone on F.Cu, net +12V
- added copper zone on F.Cu, net +BATT
- added copper zone on F.Cu, net /Synchronous buck/VOUT
- added copper zone on F.Cu, net GND
- added copper zone on F.Cu, net Net-(C10-Pad1)
- added copper zone on F.Cu, net Net-(C14-Pad2)
- added copper zone on F.Cu, net Net-(L2-Pad2)

Commit message: Update PCB
Parts:
- moved TP16 131.9 mm to (22.9, 50.8)
- moved TP17 128.7 mm to (23.9, 34.5)
- moved TP18 98.1 mm to (59.2, 6.10)
- moved TP19 88.4 mm to (68.3, 6.10)
- moved TP15 73.1 mm to (74.7, 31.0)
- moved TP20 65.0 mm to (82.0, 31.0)
- moved R18 52.4 mm to (84.2, 26.2), turned to 180 degrees
- moved R17 52.3 mm to (84.2, 24.1), turned to 180 degrees
- moved J9 52.3 mm to (89.9, 25.1)
- moved TP12 45.4 mm to (68.1, 22.9)
- moved TP13 38.7 mm to (53.6, 22.9)
- moved C1 34.3 mm to (68.2, 33.7)
- moved C19 34.3 mm to (73.7, 14.7)
- moved C2 34.3 mm to (68.2, 35.6)
- moved C20 34.3 mm to (79.0, 14.7)
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Connections:
- TP12 pad 1: SYNC_ISEN -> SYNC_ISENS
- U5 pad 10: SYNC_ISEN -> SYNC_ISENS
Routing:
- net +12V: track 3.67 -> 41.5 mm, vias 0 -> 4
- net SYNC_ISENS: track 7.95 -> 40.0 mm, vias 0 -> 3
- net Net-(Q1-Pad2): track 1.45 -> 33.1 mm, vias 1 -> 4
- net Net-(R7-Pad1): track 0.00 -> 22.3 mm, vias 0 -> 2
- net Net-(C14-Pad2): track 0.00 -> 14.4 mm, vias 0 -> 2
- net Net-(J9-Pad3): track 0.00 -> 5.02 mm
- net Net-(C11-Pad2): track 3.73 -> 8.73 mm
- net Net-(J9-Pad2): track 0.00 -> 4.99 mm
- net Net-(C14-Pad1): track 0.00 -> 4.40 mm
- net Net-(R14-Pad2): track 0.00 -> 2.18 mm
- net GND: track 40.5 -> 41.9 mm, vias 7 -> 8
Other:
- board size 127 x 63.5 mm -> 93 x 63.5 mm

Commit message: Update PCB
Parts:
- moved TP17 25.2 mm to (25.0, 9.40)
- moved TP5 24.4 mm to (5.08, 49.3)
- moved TP16 20.0 mm to (5.08, 41.7)
- moved TP2 9.99 mm to (20.1, 58.4)
- moved TP9 9.02 mm to (7.62, 26.9)
- moved TP1 3.70 mm to (13.7, 51.8)
- moved TP3 3.70 mm to (20.1, 51.8)
- moved TP4 3.07 mm to (13.7, 58.4)
- moved TP8 2.54 mm to (14.0, 19.1)
- moved TP14 2.54 mm to (7.62, 19.1)
- moved C16 1.80 mm to (34.3, 7.62)
- moved R16 1.80 mm to (39.9, 7.62)
- moved TP11 0.80 mm to (18.0, 45.2)
Connections:
- C18 pad 2: +5V -> VDD
- U5 pad 6: +5V -> VDD
Routing:
- net IO_PA0: track 34.8 -> 110.9 mm, vias 4 -> 8
- net IO_PA1: track 34.9 -> 104.3 mm, vias 2 -> 6
- net SYNC_LIN: track 7.94 -> 76.7 mm, vias 0 -> 5
- net SYNC_HIN: track 4.89 -> 70.9 mm, vias 0 -> 6
- net TCAN_nRST: track 0.00 -> 64.3 mm, vias 0 -> 5
- net SYNC_EN: track 8.46 -> 66.1 mm, vias 0 -> 4
- net +12V: track 41.5 -> 92.9 mm, vias 4 -> 6
- net VDD: track 100.7 -> 147.0 mm, vias 6 -> 8
- net /Synchronous buck/VOUT: track 0.00 -> 43.1 mm, vias 0 -> 2
- net +5V: track 12.9 -> 52.9 mm, vias 0 -> 4
- net TCAN_TS: track 31.2 -> 66.5 mm, vias 3 -> 5
- net /MCU/PC6: track 5.65 -> 40.1 mm, vias 0 -> 4
- net /MCU/PD2: track 5.13 -> 39.2 mm, vias 0 -> 4
- net GND: track 41.9 -> 9.88 mm
- net /MCU/PA3: track 49.9 -> 80.9 mm
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- added copper zone on B.Cu, net GND

Commit message: Update PCB
Other:
- board text added: "City Science Lab @ Taipei Tech ledCAN EVM DANCHOUZHOU 2022-10"
Changed lines of the file:
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@@
     (property "Sheetname" "Power")
     (attr through_hole)
-    (fp_text reference "TP17" (at 0 -2.75) (layer "F.SilkS")
+    (fp_text reference "TP17" (at 0 3.302) (layer "F.SilkS")
       (effects (font (size 1 1) (thickness 0.15)))
     )
@@
     (effects (font (size 1.5 1.5) (thickness 0.25)) (justify left mirror))
   )
+  (gr_text "City Science Lab @ Taipei Tech\nledCAN EVM\nDANCHOUZHOU 2022-10" (at 8.128 3.556) (layer "F.SilkS")
+    (effects (font (size 1 1) (thickness 0.15)) (justify left))
+  )
   (gr_text "Pmod" (at 88.265 34.925) (layer "F.SilkS")
