File: kicad/big-board/SYNC_BUCK/synchronous_buck.kicad_sch (KiCad schematic)
At the start: 22 parts

Commit message: Update schematic
Parts:
- added TP?: VFB, symbol Connector:TestPoint
- added TP? (x2): GND, symbol Connector:TestPoint
- added TP?: HIN, symbol Connector:TestPoint
- added TP?: VOUT, symbol Connector:TestPoint
- added TP?: LIN, symbol Connector:TestPoint
- added TP?: TestPoint, symbol Connector:TestPoint
- added TP?: ISEN, symbol Connector:TestPoint
- C?: value (none) -> 220nF; footprint (none) -> Capacitor_SMD:C_0603_1608Metric
- C?: value (none) -> 4.7uF; footprint (none) -> Capacitor_SMD:C_0603_1608Metric
- C?: value (none) -> 10uF; footprint (none) -> Capacitor_SMD:C_1210_3225Metric
- C?: value (none) -> 100uF; footprint (none) -> Capacitor_Tantalum_SMD:CP_EIA-7343-31_Kemet-D
- C?: value (none) -> C; footprint (none) -> Capacitor_SMD:C_0805_2012Metric_Pad1.18x1.45mm_HandSolder
- C?: footprint (none) -> Capacitor_SMD:C_0603_1608Metric
- D?: value (none) -> P4FL5.0A; footprint (none) -> Diode_SMD:D_SOD-123F
- J?: value (none) -> Conn_01x04; footprint (none) -> IO_CONN:IO_CONN
- L?: value (none) -> PM4342.472NLT; footprint (none) -> Bourns_SRP1038AA:INDPM110100X400N
- Q?: value (none) -> PSMQC092N10LS1; footprint (none) -> PANJIT_DFN:PANJIT_DFN5060-8L
- Q?: value (none) -> PSMQC076N12LS1; footprint (none) -> PANJIT_DFN:PANJIT_DFN5060-8L
- R? (x2): value (none) -> Rg; footprint (none) -> Resistor_SMD:R_0603_1608Metric
- R?: value (none) -> 2R2; footprint (none) -> Resistor_SMD:R_0805_2012Metric
- R?: value (none) -> 2K; footprint (none) -> Resistor_SMD:R_0603_1608Metric
- R?: value (none) -> 1K; footprint (none) -> Resistor_SMD:R_0603_1608Metric
- R? (x2): value (none) -> 330R; footprint (none) -> Resistor_SMD:R_0603_1608Metric
- R?: footprint (none) -> Resistor_SMD:R_Shunt_Ohmite_LVK25
- U?: value (none) -> UCC27282DRCR; footprint (none) -> Package_SON:Texas_DRC0010J_ThermalVias
- U?: value (none) -> NCS214RMUTAG; footprint (none) -> Package_DFN_QFN:UQFN-10_1.4x1.8mm_P0.4mm
Connections:
- net GND: now also TP?.1, TP?.1
- net VOUT: now also TP?.1
- net HIN renamed SYNC_HIN
- net SYNC_HIN: now also TP?.1
- net ISEN renamed SYNC_ISEN
- net SYNC_ISEN: now also TP?.1
- net ISEN_OFF renamed SENSE_OFF
- net SENSE_OFF: now also TP?.1
- net LIN renamed SYNC_LIN
- net SYNC_LIN: now also TP?.1
- net PA0 renamed IO_PA0
- net PA1 renamed IO_PA1
- net VFB renamed SYNC_VFB
- net SYNC_VFB: now also TP?.1
Other:
- note added: "Current sense offset"
- note added: "Test point"
- moved on the sheet: C?, D?, J?, L?, Q?, R?, U?

Commit message: Update schematic
Parts:
- removed TP?: TestPoint, symbol Connector:TestPoint
- added TP13: OFFSET, TestPoint:TestPoint_Keystone_5005-5009_Compact, symbol Connector:TestPoint
- added TP14: GND, TestPoint:TestPoint_Keystone_5005-5009_Compact, symbol Connector:TestPoint
- C18: renamed from C?; footprint (none) -> Capacitor_SMD:C_0603_1608Metric
- TP10, TP11, TP12, TP6, TP7, TP8, TP9: renamed from TP?; footprint (none) -> TestPoint:TestPoint_Keystone_5005-5009_Compact
- gave numbers to parts that had none: 21
Connections:
- net GND: now also TP14.1
- net SENSE_OFF: now also TP13.1
Other:
- note added: "Current sense TP"
- note removed: "Current sense offset"
- moved on the sheet: TP10, TP11, TP12, TP6, TP7, TP8, TP9

Commit message: Update PCB
Parts:
- added C20, C21: 100uF, Capacitor_Tantalum_SMD:CP_EIA-7343-31_Kemet-D, symbol Device:C_Polarized
Connections:
- net +12V: no longer U4.6 (EN)
- net GND: now also C20.2, C21.2
- net VOUT: now also C20.1, C21.1
- new net SYNC_EN: U4.6 (EN)
Other:
- moved on the sheet: D3

Commit message: Update PCB
Parts:
- C16: footprint Capacitor_SMD:C_0805_2012Metric_Pad1.18x1.45mm_HandSolder -> Capacitor_SMD:C_1206_3216Metric
- R16: footprint Resistor_SMD:R_0805_2012Metric -> Resistor_SMD:R_1206_3216Metric_Pad1.30x1.75mm_HandSolder
Changed lines of the file:
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@@
       (effects (font (size 1.27 1.27)) (justify left))
     )
-    (property "Footprint" "Resistor_SMD:R_0805_2012Metric" (id 2) (at 156.972 127 90)
+    (property "Footprint" "Resistor_SMD:R_1206_3216Metric_Pad1.30x1.75mm_HandSolder" (id 2) (at 156.972 127 90)
       (effects (font (size 1.27 1.27)) hide)
     )
@@
       (effects (font (size 1.27 1.27)) (justify left))
     )
-    (property "Footprint" "Capacitor_SMD:C_0805_2012Metric_Pad1.18x1.45mm_HandSolder" (id 2) (at 159.7152 143.51 0)
+    (property "Footprint" "Capacitor_SMD:C_1206_3216Metric" (id 2) (at 159.7152 143.51 0)
       (effects (font (size 1.27 1.27)) hide)
     )

Commit message: Update PCB
Connections:
- net at L2.2: now also R19.3; no longer R19.1
- net at U5.4 (-IN), U5.5 (-IN): now also R19.1; no longer R19.3
Changed lines of the file:
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@@
   )
   (symbol (lib_id "Device:R_Shunt") (at 187.96 120.65 90) (unit 1)
-    (in_bom yes) (on_board yes) (fields_autoplaced)
-    (property "Reference" "R19" (id 0) (at 187.96 124.46 90))
-    (property "Value" "LVK25R001FER" (id 1) (at 187.96 127 90))
-    (property "Footprint" "Resistor_SMD:R_Shunt_Ohmite_LVK25" (id 2) (at 187.96 122.428 90)
+    (in_bom yes) (on_board yes)
+    (property "Reference" "R19" (id 0) (at 187.96 120.65 90))
+    (property "Value" "LVK25R001FER" (id 1) (at 190.5 120.65 90))
+    (property "Footprint" "Resistor_SMD:R_Shunt_Ohmite_LVK25" (id 2) (at 186.182 120.65 90)
       (effects (font (size 1.27 1.27)) hide)
     )
@@
       (effects (font (size 1.27 1.27)) hide)
     )
+    (pin "2")
     (pin "1")
-    (pin "2")
     (pin "3")
     (pin "4")

Commit message: Update PCB
Connections:
- net SYNC_ISEN renamed SYNC_ISENS
Changed lines of the file:
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@@
     )
   )
-  (global_label "SYNC_ISEN" (shape output) (at 247.65 45.72 0) (fields_autoplaced)
+  (global_label "SYNC_ISENS" (shape output) (at 247.65 45.72 0) (fields_autoplaced)
     (effects (font (size 1.27 1.27)) (justify left))
-    (property "Intersheet References" "${INTERSHEET_REFS}" (id 0) (at 260.2231 45.6406 0)
+    (property "Intersheet References" "${INTERSHEET_REFS}" (id 0) (at 261.4326 45.6406 0)
       (effects (font (size 1.27 1.27)) (justify left) hide)
     )
@@
       (effects (font (size 1.27 1.27)) hide)
     )
-    (pin "2")
-    (pin "1")
+    (pin "1")
+    (pin "2")
     (pin "3")
     (pin "4")

Commit message: Update PCB
Connections:
- net +5V renamed VDD
Changed lines of the file:
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@@
-    (pin "1")
-  )
-  (symbol (lib_id "power:+5V") (at 213.36 81.28 0) (unit 1)
-    (in_bom yes) (on_board yes)
-    (property "Reference" "#PWR061" (id 0) (at 213.36 85.09 0)
-      (effects (font (size 1.27 1.27)) hide)
-    )
-    (property "Value" "+5V" (id 1) (at 213.741 76.8858 0))
-    (property "Footprint" "" (id 2) (at 213.36 81.28 0)
-      (effects (font (size 1.27 1.27)) hide)
-    )
-    (property "Datasheet" "" (id 3) (at 213.36 81.28 0)
-      (effects (font (size 1.27 1.27)) hide)
-    )
     (pin "1")
   )
@@
       (effects (font (size 1.27 1.27)) hide)
     )
+    (pin "1")
+  )
+  (symbol (lib_id "power:VDD") (at 213.36 81.28 0) (unit 1)
+    (in_bom yes) (on_board yes) (fields_autoplaced)
+    (property "Reference" "#PWR?" (id 0) (at 213.36 85.09 0)
+      (effects (font (size 1.27 1.27)) hide)
+    )
+    (property "Value" "VDD" (id 1) (at 213.36 76.2 0))
+    (property "Footprint" "" (id 2) (at 213.36 81.28 0)
+      (effects (font (size 1.27 1.27)) hide)
+    )
+    (property "Datasheet" "" (id 3) (at 213.36 81.28 0)
+      (effects (font (size 1.27 1.27)) hide)
+    )
